Commit message: 111

File: src/ros2_foundry_description/urdf/monolithic_bot.urdf (robot description, URDF)
Before this commit: robot foundry_bot, 18 links, 17 joints
Joints:
- joint left_wheel_joint: limit (none) -> lower=-10000 upper=10000 effort=100 velocity=100; type continuous -> revolute
- joint right_wheel_joint: limit (none) -> lower=-10000 upper=10000 effort=100 velocity=100; type continuous -> revolute
